Commit message: teleop kinda functional

File: giraffe.urdf (robot description, URDF)
Before this commit: robot giraffe, 7 links, 6 joints
Links:
- link base_link: mass 0.812217234610215 -> 0.8122108919622869; geometry collision mesh filename=package://giraffe_description/meshes/base_link.stl scale=0.001 0.001 0.001; visual mesh filename=package://giraffe_description/meshes/base_link.stl scale=0.001 0.001 0.001
- link elbow: geometry collision mesh filename=package://giraffe_description/meshes/elbow.stl scale=0.001 0.001 0.001; visual mesh filename=package://giraffe_description/meshes/elbow.stl scale=0.001 0.001 0.001
- link gripper: geometry collision mesh filename=package://giraffe_description/meshes/gripper.stl scale=0.001 0.001 0.001; visual mesh filename=package://giraffe_description/meshes/gripper.stl scale=0.001 0.001 0.001
- link shoulder_lift: geometry collision mesh filename=package://giraffe_description/meshes/shoulder_lift.stl scale=0.001 0.001 0.001; visual mesh filename=package://giraffe_description/meshes/shoulder_lift.stl scale=0.001 0.001 0.001
- link shoulder_pan: geometry collision mesh filename=package://giraffe_description/meshes/shoulder_pan.stl scale=0.001 0.001 0.001; visual mesh filename=package://giraffe_description/meshes/shoulder_pan.stl scale=0.001 0.001 0.001
- link wrist_1: mass 0.11585466541730398 -> 0.11585466541730399; geometry collision mesh filename=package://giraffe_description/meshes/wrist_1.stl scale=0.001 0.001 0.001; visual mesh filename=package://giraffe_description/meshes/wrist_1.stl scale=0.001 0.001 0.001
- link wrist_2: mass 0.20479740953235445 -> 0.20479740953235442; geometry collision mesh filename=package://giraffe_description/meshes/wrist_2.stl scale=0.001 0.001 0.001; visual mesh filename=package://giraffe_description/meshes/wrist_2.stl scale=0.001 0.001 0.001
Joints:
- joint base_link_shoulder_pan_joint: axis -2.465190328815662e-32 7.92896871208326e-16 1.0 -> -4.930380657631324e-32 2.37251531204244e-15 1.0; origin xyz=-0.007481813113703827 -0.18092165633421572 -0.051176553314811093 rpy=1.3902260885354034e-15 1.2005791989029008e-16 -0.0007586542251338113 -> xyz=0.09891995753862716 -0.00013303607482287617 0.05455000000000001 rpy=3.189786117866041e-15 3.393805650568627e-16 -0.0007586542251351899
- joint elbow_wrist_1_joint: axis -0.0007583461697307804 -1.8676166605626716e-13 -0.9999998631005341 -> -0.9999998631005341 -1.23112379231774e-10 0.0007583461697307804; limit lower=-3.368485 upper=0.261799 effort=1000000 velocity=1000000 -> lower=-1.797689 upper=1.797689 effort=1000000 velocity=1000000; origin xyz=-0.12026017684124206 -0.002215789985019754 -0.037616306707671 rpy=1.878793372233325e-13 2.512616851854867e-14 -2.476481313343611e-10 -> xyz=-0.03761630670794674 -0.0022157899953267803 0.12026017684096592 rpy=1.8787933722333255e-13 2.512616851854867e-14 -2.476481313343611e-10
- joint shoulder_lift_elbow_joint: axis 3.456292375562768e-07 -9.452259649568135e-14 1.0000002880403989 -> 1.0000002880403989 -1.245357002578147e-10 -3.456292375562768e-07; limit lower=-1.53589 upper=1.745329 effort=1000000 velocity=1000000 -> lower=-1.53589 upper=1.780236 effort=1000000 velocity=1000000; origin xyz=-0.025196435278486345 0.10949146000520331 -0.037893485524666634 rpy=3.1415926535895418 2.2650067565861562e-14 -3.312801036946675e-10 -> xyz=0.037893485547286214 0.10949145999216181 -0.025196435301140276 rpy=3.1415926535895418 2.265006756586156e-14 -3.3128010369466755e-10
- joint shoulder_pan_shoulder_lift_joint: axis 0.000758654152361514 -3.814002872675493e-38 0.9999997122218974 -> -0.9999997122218972 2.0674449877203995e-10 0.0007586541523615138; limit lower=-0.785398 upper=1.644158 effort=1000000 velocity=1000000 -> lower=-0.785398 upper=1.658063 effort=1000000 velocity=1000000; origin xyz=-0.01894466000000003 0.02571941000000001 0.01737606999999998 rpy=1.5707963267950535 -2.0674523217214331e-10 -1.5715549810200329 -> xyz=0.02571940999999997 0.018944660000000037 0.017376069999999952 rpy=1.5707963267950535 -2.0674681179012968e-10 -1.5715549810200329
- joint wrist_1_wrist_2_joint: axis -1.3510287936481513e-07 1.2304131739319882e-05 1.0000004491016943 -> -0.9999449329225374 0.006662002215913354 -0.008132268196377131; origin xyz=-0.00017835491299077687 0.06033854999998056 0.027120202494905085 rpy=-3.049102007927164 1.5625820319968764 -1.4783560893203032 -> xyz=0.027165827341760113 -0.00019891999664992 0.06031796682590525 rpy=-3.049102007927164 1.5625820319968764 -1.4783560893203032
- joint wrist_2_gripper_joint: axis -0.0015173474686189948 -5.3999999838870086e-05 0.9999984389196113 -> -0.007420635544791429 -0.0007590000001611277 -0.9999726580742655; limit lower=-0.174533 upper=1.570796 effort=1000000 velocity=1000000 -> lower=0.0 upper=1.570796 effort=1000000 velocity=1000000; origin xyz=0.02541041108611911 0.01946328617934281 0.017249861388580517 rpy=-1.5708498378135036 -0.008179184380179302 0.0007586796016247197 -> xyz=-0.017171676526959914 -0.019310353391698003 -0.025579471562416883 rpy=-1.5708498378135036 -0.0081791843801793 0.0007586796016247204

Commit message: calib, roll, pitch fixed

File: giraffe.urdf (robot description, URDF)
Before this commit: robot giraffe, 7 links, 6 joints
Joints:
- joint shoulder_lift_elbow_joint: origin xyz=0.037893485547286214 0.10949145999216181 -0.025196435301140276 rpy=3.1415926535895418 2.265006756586156e-14 -3.3128010369466755e-10 -> xyz=0.037893485547286214 0.10949145999216181 -0.025196435301140276 rpy=3.1415926535895418 2.265006756586156e-14 -3.364010369466755e-10
- joint shoulder_pan_shoulder_lift_joint: axis -0.9999997122218972 2.0674449877203995e-10 0.0007586541523615138 -> -0.9999997122218972 2.0674449874803995e-10 0.0007586541523615138
- joint wrist_2_gripper_joint: origin xyz=-0.017171676526959914 -0.019310353391698003 -0.025579471562416883 rpy=-1.5708498378135036 -0.0081791843801793 0.0007586796016247204 -> xyz=-0.017171676526959914 -0.019310353391698003 -0.025579471562416883 rpy=-1.5708498378135036 -0.0081791843801793 0.0007586796016244804
